File: SIEBOT2/STM32.sch (KiCad schematic (older format))
At the start: 22 parts

Commit message: Added some fixes from AndroidStamp
Parts:
- removed SW?: SW_PUSH, symbol SW_PUSH
Connections:
- net labels added: STM32_NRST, TIM16_BKIN, TIM16_CH1, TIM17_CH1, TIM2_CH1_ETR, TIM2_CH2

Commit message: Added power dc-dc, fixed stm32 control pins
Parts:
- removed K? (x2): CONN_3, symbol CONN_3
- gave numbers to parts that had none: 19
Connections:
- net labels added: STM32_ADC[0..15], STM32_BOOT0, STM32_BOOT1, STM32_P[A13..E15]
- net labels removed: STM32_ADC, STM32_GPIOs
- wire segments 162 -> 157
- no-connect marks 6 -> 2
Other:
- moved on the sheet: RP1

Commit message: STM32 connection fixes + various fixes
Parts:
- added D1: LED, symbol LED
- added R3: 1k, symbol R
Connections:
- net labels added: STM32_GPIO0, STM32_GPIO1, STM32_GPIO10, STM32_GPIO11, STM32_GPIO12, STM32_GPIO13, STM32_GPIO14, STM32_GPIO15, STM32_GPIO16, STM32_GPIO17, STM32_GPIO18, STM32_GPIO19, STM32_GPIO2, STM32_GPIO20, STM32_GPIO21, STM32_GPIO22, STM32_GPIO23, STM32_GPIO24, STM32_GPIO25, STM32_GPIO3, STM32_GPIO4, STM32_GPIO5, STM32_GPIO6, STM32_GPIO7, STM32_GPIO8, STM32_GPIO9, STM32_GPIO[0..25], TIM0, TIM1, TIM10, TIM11, TIM12, TIM13, TIM14, TIM15, TIM16, TIM17, TIM18, TIM19, TIM2, TIM20, TIM21, TIM22, TIM23, TIM3, TIM4, TIM5, TIM6, TIM7, TIM8, TIM9, TIM[00..23]
- net labels removed: STM32_PA13, STM32_PA14, STM32_PB4, STM32_PC10, STM32_PC11, STM32_PC12, STM32_PD0, STM32_PD1, STM32_PD10, STM32_PD11, STM32_PD3, STM32_PD4, STM32_PD7, STM32_PE1, STM32_PE10, STM32_PE12, STM32_PE14, STM32_PE15, STM32_PE2, STM32_PE3, STM32_PE4, STM32_PE5, STM32_PE6, STM32_PE7, STM32_PE8, STM32_PE9, STM32_P[A13..E15], STM32_TIMs
- wire segments 157 -> 161
Other:
- note added: "TEST LED (Hello World intended)"
- moved on the sheet: X2
