File: SIEBOT2/i.MX233.sch (KiCad schematic (older format))
At the start: 72 parts, among them IC1 iMX233, J1 MICROSD, P1 CONN_8X2, P2 CONN_12X2, P3 CONN_5X2, P5 CONN_4, P6 CONN_2X2, Q1 MMDT3904, SW1 SW_PUSH, SW2 SW_PUSH, SW3 SW_PUSH, X1 24 MHz

Commit message: Added some fixes from AndroidStamp
Parts:
- removed P6: CONN_2X2, symbol CONN_2X2
- removed R26: 10K, symbol R
- removed R27: 22, symbol R
- added C? (x5): 0.1uF, symbol C
- added D? (x4): LED, symbol LED
- added P?: CONN_2X2, symbol CONN_2X2
- added P?: CONN_4, symbol CONN_4
- added R? (x4): 1k, symbol R
- added R?: 22, symbol R
- added R?: 10K, symbol R
- added R?: 47k, symbol R
- added U?: ADM3101E, symbol ADM3101E
Connections:
- net labels added: LCD_D04, LCD_D05, LCD_D06, LCD_D07, PMW0, PMW1, RX, TX
- wire segments 334 -> 374
- no-connect marks 17 -> 18
Other:
- note added: "TRANCEIVER_RS232/CMOS"
- note added: "UART CONNECTOR"
- moved on the sheet: C57, C60, J1, P1, P2, P3, P5, Q1, R10, R11, R12, R13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

Commit message: Added power dc-dc, fixed stm32 control pins
Parts:
- removed D?: LED, symbol LED
- removed P?: CONN_2X2, symbol CONN_2X2
- removed R?: 1k, symbol R
- gave numbers to parts that had none: 16
- renumbered C22 to C28, C23 to C29, C24 to C30, C52 to C31, C53 to C32, C26 to C33, C25 to C34, C28 to C35, C27 to C36, C29 to C37, C30 to C38, C31 to C39, C32 to C40, C34 to C41, C35 to C42, C36 to C43, C37 to C44, C38 to C45, C39 to C46, C40 to C47, C41 to C48, C42 to C49, C43 to C50, C44 to C51, C45 to C52, C46 to C53, C47 to C54, C48 to C55, C49 to C56, C50 to C57, C51 to C58, C56 to C59, C57 to C60, C60 to C61, D1 to D3, L1 to L2, P5 to P10, P3 to P7, P1 to P8, P2 to P9, R1 to R17, R2 to R18, R3 to R20, R4 to R23, R13 to R24, R5 to R26, R6 to R27, R16 to R28, R10 to R29, R11 to R31, R12 to R32, R14 to R33, R15 to R34, R17 to R35, R18 to R36, R19 to R37, R20 to R38, R21 to R39, RP5 to RP2, SW3 to SW1, SW1 to SW2, SW2 to SW3, X1 to X3
Connections:
- net labels added: 3V3, 5V
- net labels removed: GNDPWR, VBUS, VBUS_HOST
- wire segments 374 -> 370
- no-connect marks 18 -> 14
Other:
- note added: "STM32 INTERFACE"
- note removed: "Power Supply"
- moved on the sheet: C29, C33, C35, C37, C60, J1, P10, P11, R23, R25, R26, R27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

Commit message: STM32 connection fixes + various fixes
Parts:
- removed P7: CONN_5X2, symbol CONN_5X2
- removed R33: 47K, symbol R
- added JP3: JUMPER, symbol JUMPER
- added L3: HZ0805D152R-10 (1500 ohm), symbol INDUCTOR
- added P8: CONN_4X2, symbol CONN_4X2
- added R36: 47K, symbol R
- R25: renamed from R24; value 1K -> 47K
- R29: renamed from R28; value 1K -> 47K
- R35: value 1.2K -> 47K
- R37: renamed from R36; value 1.2K -> 10K
- R38: renamed from R37; value 1.2K -> 10K
- R39: renamed from R38; value 1.2K -> 10K
- R40: renamed from R39; value 1.2K -> 10K
- renumbered D2 to D3, D3 to D4, D4 to D5, D5 to D6, P9 to P10, P10 to P11, P11 to P12, P8 to P9, R17 to R18, R18 to R19, R19 to R20, R20 to R21, R21 to R22, R22 to R23, R23 to R24, R25 to R26, R26 to R27, R27 to R28, R29 to R32, R32 to R33, R40 to R41
Connections:
- net labels added: SD_DAT3
- net labels removed: PMW0, PMW1
- wire segments 370 -> 376
Other:
- note added: "HAY QUE VERIFICAR ESTO, LA CORRIENTE MÁXIMA ES COMPARTIDA CON LOS \nREGULADORES DE VDDD, VDDA Y VDDM, ASÍ QUE PROBABLEMENTE CON LA \nBATERÍA DESCARGADA HAYA PROBLEMAS DE ALIMENTACIÓN TANTO EN \nEL iMX COMO EN EL STM32"
- moved on the sheet: R31, R32, R33, R34, R37, R38, R39, R40

Commit message: iMX233 boot modes circuit modified
Parts:
- removed P8: CONN_4X2, symbol CONN_4X2
- removed R37, R40: 10K, symbol R
- added P?: CONN_2X2, symbol CONN_2X2
